File: pcb/cave.kicad_pcb (KiCad board)
At the start: 2 copper layers, 46.5 x 65 mm, 31 parts, among them J1 Raspberry_Pi_2_3, J2 PIRsensor, J3 PWR, J4 RelayOutput, U1 LM2576S-5, U2 DS18B20, U3 LM386

Commit message: fixed rectifier layout and PIR position
Parts:
- C7: footprint Capacitor_THT:CP_Radial_D7.5mm_P2.50mm -> Capacitor_THT:CP_Radial_D10.0mm_P2.50mm
- J2: footprint Connector_JST:JST_PH_B3B-PH-K_1x03_P2.00mm_Vertical -> Connector_PinHeader_2.54mm:PinHeader_1x03_P2.54mm_Vertical
- moved J2 15.2 mm to (158.2, 138.5), turned to 90 degrees
- moved C7 0.17 mm to (176.8, 94.0)
Connections:
- C6 pad 1: +24V -> Net-(C6-Pad1)
- D5 pad 1: +24V -> Net-(C6-Pad1)
- D6 pad 1: +24V -> Net-(C6-Pad1)
- U1 pad 1: +24V -> Net-(C6-Pad1)
Routing:
- net +24V: track 51.0 -> 16.1 mm
- net Net-(C6-Pad1): track 0.00 -> 34.2 mm
- net GND: track 202.3 -> 219.4 mm
- net /PIR: track 35.5 -> 51.6 mm
- net +5V: track 103.1 -> 118.5 mm
- net -24V: track 18.5 -> 19.7 mm, vias 1 -> 0
Other:
- board text added: "Cave V1.1"
- board text removed: "Cave V1"

Commit message: added more labels to pcb
Other:
- board text added: "5V"
- board text added: "GND"
Changed lines of the file:
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@@
-(kicad_pcb (version 20171130) (host pcbnew 5.0.1)
+(kicad_pcb (version 20171130) (host pcbnew 5.1.4)
   (general
     (thickness 1.6)
-    (drawings 5)
+    (drawings 11)
     (tracks 265)
     (zones 0)
@@
     (zone_45_only no)
     (trace_min 0.2)
-    (segment_width 0.2)
-    (edge_width 0.2)
     (via_size 0.8)
     (via_drill 0.4)
@@
     (uvia_min_size 0.2)
     (uvia_min_drill 0.1)
+    (edge_width 0.2)
+    (segment_width 0.2)
     (pcb_text_width 0.3)
     (pcb_text_size 1.5 1.5)
@@
     )
   )
+  (gr_text 5V (at 198.52 133.73 90) (layer F.SilkS)
+    (effects (font (size 1 1) (thickness 0.25)))
+  )
+  (gr_text GND (at 198.52 120.88 90) (layer F.SilkS)
+    (effects (font (size 1 1) (thickness 0.25)))
+  )
+  (gr_text GND (at 182.56 134.06) (layer B.SilkS)
+    (effects (font (size 1 1) (thickness 0.25)) (justify mirror))
+  )
+  (gr_text 5V (at 190.1 83.02) (layer B.SilkS)
+    (effects (font (size 1 1) (thickness 0.25)) (justify mirror))
+  )
+  (gr_text GND (at 182.34 133.72) (layer F.SilkS)
+    (effects (font (size 1 1) (thickness 0.25)))
+  )
+  (gr_text 5V (at 189.82 82.62) (layer F.SilkS)
+    (effects (font (size 1 1) (thickness 0.25)))
+  )
   (gr_text "Cave V1.1" (at 176 138.5) (layer F.SilkS)
     (effects (font (size 1.5 1.5) (thickness 0.3)))
@@
   (segment (start 156.17 81.87) (end 156.17 82.87) (width 0.25) (layer B.Cu) (net 9))
   (segment (start 159.54 78.5) (end 156.17 81.87) (width 0.25) (layer B.Cu) (net 9))
-  (segment (start 173.225001 86.724999) (end 168 91.95) (width 0.25) (layer B.Cu) (net 55))
-  (segment (start 173.225001 83.512499) (end 173.225001 86.724999) (width 0.25) (layer B.Cu) (net 55))
-  (segment (start 177.7375 79) (end 173.225001 83.512499) (width 0.25) (layer B.Cu) (net 55))
-  (segment (start 178 79) (end 177.7375 79) (width 0.25) (layer B.Cu) (net 55))
-  (segment (start 168 93) (end 168 91.95) (width 0.25) (layer B.Cu) (net 55))
   (segment (start 161.580002 87.160002) (end 163.795001 89.375001) (width 0.25) (layer B.Cu) (net 9))
   (segment (start 161.580002 87.130002) (end 157.32 82.87) (width 0.25) (layer B.Cu) (net 9))
@@
   (segment (start 173.15 78) (end 175.85 80.7) (width 0.25) (layer F.Cu) (net 54))
   (segment (start 172 78) (end 173.15 78) (width 0.25) (layer F.Cu) (net 54))
+  (segment (start 173.225001 86.724999) (end 168 91.95) (width 0.25) (layer B.Cu) (net 55))
+  (segment (start 173.225001 83.512499) (end 173.225001 86.724999) (width 0.25) (layer B.Cu) (net 55))
+  (segment (start 177.7375 79) (end 173.225001 83.512499) (width 0.25) (layer B.Cu) (net 55))
+  (segment (start 178 79) (end 177.7375 79) (width 0.25) (layer B.Cu) (net 55))
+  (segment (start 168 93) (end 168 91.95) (width 0.25) (layer B.Cu) (net 55))
   (segment (start 156.175001 90.525001) (end 156.175001 92.625001) (width 0.25) (layer B.Cu) (net 55))
   (segment (start 156.175001 89.375001) (end 156.175001 90.525001) (width 0.25) (layer B.Cu) (net 55))
